File: PCB/Blinker.kicad_pcb (KiCad board)
At the start: 2 copper layers, 100 x 100 mm, 69 parts, among them J1 Conn_01x02_Pin, U1 4017, U2 NE555P

Commit message: Done
Parts:
- added G***: LOGO, kicadlogos:communism, F.Cu at (117.0, 118.0)
- added G***: LOGO, kicadlogos:communism, F.Cu at (119.0, 68.0)
- added G***: LOGO, kicadlogos:communism, F.Cu at (167.0, 119.0)
- added G***: LOGO, kicadlogos:Commiebig, F.Cu at (151.0, 99.0)
- added G***: LOGO, kicadlogos:communism, F.Cu at (169.0, 69.0)
